File: hardware/pcb/pcb.kicad_pcb (KiCad board)
At the start: 2 copper layers, 4 parts, among them U101 LTC6811HG-1#3ZZTRPBF, U102 HCZZ0520-13, U103 HCZZ0520-13, U104 ESP32-C3

Commit message: re writing the code for better optimization
Parts:
- removed U101: LTC6811HG-1#3ZZTRPBF, easyeda2kicad:SSOP-48_L12.8-W5.3-P0.50-LS7.8-BL
- added C101: 0.1uF, PCM_Capacitor_SMD_AKL:C_0402_1005Metric, B.Cu at (87.2, 142.3)
- added C102: 0.1uF, PCM_Capacitor_SMD_AKL:C_0402_1005Metric, B.Cu at (86.0, 142.3)
- added C103: 0.1uF, PCM_Capacitor_SMD_AKL:C_0402_1005Metric, B.Cu at (109.4, 133.3)
- added C104: 0.1uF, PCM_Capacitor_SMD_AKL:C_0402_1005Metric, B.Cu at (95.5, 138.8)
- added C105: 0.1uF, PCM_Capacitor_SMD_AKL:C_0402_1005Metric, B.Cu at (117.4, 139.3)
- added C106: 1uF, PCM_Capacitor_SMD_AKL:C_0402_1005Metric, B.Cu at (106.3, 129.1)
- added C107: 0.1uF, PCM_Capacitor_SMD_AKL:C_0402_1005Metric, B.Cu at (106.3, 131.2)
- added C108: 10uF, PCM_Capacitor_SMD_AKL:C_0402_1005Metric, B.Cu at (106.3, 133.3)
- added C109: 10nF, PCM_Capacitor_SMD_AKL:C_0402_1005Metric, B.Cu at (92.4, 137.2)
- added C110: 1uF, PCM_Capacitor_SMD_AKL:C_0402_1005Metric, B.Cu at (92.4, 136.0)
- added L101: 27nH, Inductor_SMD:L_1206_3216Metric_Pad1.22x1.90mm_HandSolder, B.Cu at (118.5, 141.4)
- added L102: RFECA3216060A1T, easyeda2kicad:ANT-SMD_L3.1-W1.6, B.Cu at (123.7, 141.4)
- added L103: 2.0nH, Inductor_SMD:L_1206_3216Metric_Pad1.22x1.90mm_HandSolder, B.Cu at (95.7, 142.0)
- added U105: ESP32-C3, easyeda2kicad:QFN-32_L5.0-W5.0-P0.50-TL-EP3.7, B.Cu at (91.2, 141.1)
- U102: value HCZZ0520-13 -> BQ7694003DBTR; footprint easyeda2kicad:CONN-SMD_13P-P2.50_HCZZ0520-13 -> easyeda2kicad:TSSOP-44_L10.0-W4.4-P0.50-LS6.4-BL-EP; moved to B.Cu
- U104: value ESP32-C3 -> HCZZ0520-13; footprint Package_DFN_QFN:QFN-32-1EP_5x5mm_P0.5mm_EP3.7x3.7mm -> easyeda2kicad:CONN-SMD_13P-P2.50_HCZZ0520-13
- moved U103 56.1 mm to (174.2, 129.0), turned to -90 degrees
- moved U102 44.3 mm to (162.2, 116.7), turned to 90 degrees
- moved U104 29.3 mm to (188.2, 129.0), turned to 90 degrees
Connections:
- U102 pad 3: unconnected-(U102-Pad3) -> GND
- U102 pad 4: unconnected-(U102-Pad4) -> I2C_SDA
- U102 pad 5: unconnected-(U102-Pad5) -> I2C_SCL
- U103 pad 14: unconnected-(U103-Pad14) -> GND
- U103 pad 15: unconnected-(U103-Pad15) -> GND
- U104 pad 14: unconnected-(U104-GPIO8-Pad14) -> GND
- U104 pad 15: unconnected-(U104-GPIO9-Pad15) -> GND
- U104 pad 2: Net-(U104-VDD3P3-Pad2) -> unconnected-(U104-Pad2)
- U104 pad 3: Net-(U104-VDD3P3-Pad2) -> unconnected-(U104-Pad3)

Commit message: readme done and eveyrthing done
Parts:
- removed C101, C102, C103, C104, C105, C107: 0.1uF, PCM_Capacitor_SMD_AKL:C_0402_1005Metric
- removed C106, C110: 1uF, PCM_Capacitor_SMD_AKL:C_0402_1005Metric
- removed C108: 10uF, PCM_Capacitor_SMD_AKL:C_0402_1005Metric
- removed C109: 10nF, PCM_Capacitor_SMD_AKL:C_0402_1005Metric
- removed L101: 27nH, Inductor_SMD:L_1206_3216Metric_Pad1.22x1.90mm_HandSolder
- removed L102: RFECA3216060A1T, easyeda2kicad:ANT-SMD_L3.1-W1.6
- removed L103: 2.0nH, Inductor_SMD:L_1206_3216Metric_Pad1.22x1.90mm_HandSolder
- removed U105: ESP32-C3, easyeda2kicad:QFN-32_L5.0-W5.0-P0.50-TL-EP3.7
- added C111: 1uF, Capacitor_SMD:C_0402_1005Metric, B.Cu at (170.3, 144.4)
- added C112: 1uF, Capacitor_SMD:C_0402_1005Metric, B.Cu at (171.0, 133.5)
- added C113: 1uF, Capacitor_SMD:C_0402_1005Metric, B.Cu at (170.0, 133.5)
- added C114: 47nF, Capacitor_SMD:C_0402_1005Metric, B.Cu at (170.3, 135.7)
- added C118: 1uF, PCM_Capacitor_SMD_AKL:C_0805_2012Metric, B.Cu at (191.9, 134.3)
- added C119: 1uF, PCM_Capacitor_SMD_AKL:C_0805_2012Metric, B.Cu at (192.9, 123.3)
- added C120: 0.1uF, PCM_Capacitor_SMD_AKL:C_0402_1005Metric, B.Cu at (173.3, 127.6)
- added C121: 1uF, PCM_Capacitor_SMD_AKL:C_0402_1005Metric, B.Cu at (173.3, 126.4)
- added C122: 0.1uF, PCM_Capacitor_SMD_AKL:C_0402_1005Metric, B.Cu at (173.3, 133.0)
- added C123: 0.1uF, PCM_Capacitor_SMD_AKL:C_0402_1005Metric, B.Cu at (170.4, 125.7)
- added C124: 0.1uF, PCM_Capacitor_SMD_AKL:C_0402_1005Metric, B.Cu at (170.5, 126.8)
- added C125: 10nF, PCM_Capacitor_SMD_AKL:C_0402_1005Metric, B.Cu at (170.5, 128.0)
- added C126: 1uF, PCM_Capacitor_SMD_AKL:C_0402_1005Metric, B.Cu at (170.0, 121.2)
- added LED101: LED25, PCM_LED_SMD_AKL:LED_0603_1608Metric, F.Cu at (171.0, 150.6)
- added LED102: LED50, PCM_LED_SMD_AKL:LED_0603_1608Metric, F.Cu at (173.4, 150.6)
- added LED103: LED75, PCM_LED_SMD_AKL:LED_0603_1608Metric, F.Cu at (175.8, 150.6)
- added LED104: LED100, PCM_LED_SMD_AKL:LED_0603_1608Metric, F.Cu at (178.2, 150.6)
- added LED105: STATUS, PCM_LED_SMD_AKL:LED_0603_1608Metric, F.Cu at (180.6, 150.6)
- added R101: 75, PCM_Resistor_SMD_AKL:R_0402_1005Metric, B.Cu at (171.0, 150.6)
- added R102: 75, PCM_Resistor_SMD_AKL:R_0402_1005Metric, B.Cu at (173.4, 150.6)
- added R103: 75, PCM_Resistor_SMD_AKL:R_0402_1005Metric, B.Cu at (175.8, 150.6)
- added R104: 75, PCM_Resistor_SMD_AKL:R_0402_1005Metric, B.Cu at (178.2, 150.6)
- added R105: 75, PCM_Resistor_SMD_AKL:R_0402_1005Metric, B.Cu at (180.6, 150.6)
- added R106: 100R, PCM_Resistor_SMD_AKL:R_0402_1005Metric, B.Cu at (177.3, 146.7)
- added R107: 4.7k, PCM_Resistor_SMD_AKL:R_0402_1005Metric, B.Cu at (170.0, 117.0)
- added R108: 4.7k, PCM_Resistor_SMD_AKL:R_0402_1005Metric, B.Cu at (170.0, 119.0)
- added R109: 10k, PCM_Resistor_SMD_AKL:R_0402_1005Metric, B.Cu at (170.0, 123.5)
- added R110: 10k, PCM_Resistor_SMD_AKL:R_0402_1005Metric, B.Cu at (191.4, 120.7)
- added RN101: 100R, PCM_Resistor_SMD_AKL:R_Array_Convex_4x0402, B.Cu at (184.9, 146.7)
- added RN102: 100R, PCM_Resistor_SMD_AKL:R_Array_Convex_4x0402, B.Cu at (182.1, 146.7)
- added RN103: 100R, PCM_Resistor_SMD_AKL:R_Array_Convex_4x0402, B.Cu at (179.3, 146.7)
- added U101: BQ7695202PFBR, easyeda2kicad:TQFP-48_L7.0-W7.0-P0.50-LS9.0-TL, B.Cu at (174.6, 139.8)
- added U106: ZXTR2012P5-13, easyeda2kicad:POWERDI-5_L5.4-W4.0-LS6.5-RD, B.Cu at (191.9, 130.2)
- added U107: ESP32-C3-WROOM-02U, RF_Module:ESP32-C3-WROOM-02U, B.Cu at (180.9, 117.2)
- U102: value BQ7694003DBTR -> MIC5219-3.3YM5; footprint easyeda2kicad:TSSOP-44_L10.0-W4.4-P0.50-LS6.4-BL-EP -> easyeda2kicad:SOT-23-5_L3.0-W1.7-P0.95-LS2.8-TL
- U103: value HCZZ0520-13 -> INPUT
- U104: value HCZZ0520-13 -> OUTPUT
- moved U102 17.6 mm to (173.3, 130.3), turned to -90 degrees
- moved U104 1.35 mm to (189.6, 129.1)
Connections:
- U102 pad 1: unconnected-(U102-DSG-Pad1) -> 12V
- U102 pad 2: unconnected-(U102-CHG-Pad2) -> GND
- U102 pad 3: GND -> 12V
- U102 pad 4: I2C_SDA -> unconnected-(U102-BYP-Pad4)
- U102 pad 5: I2C_SCL -> VCC_3V3
- U103 pad 1: unconnected-(U103-Pad1) -> Net-(RN101A-R1.2)
- U103 pad 10: unconnected-(U103-Pad10) -> Net-(RN103B-R2.2)
- U103 pad 11: unconnected-(U103-Pad11) -> Net-(RN103C-R3.2)
- U103 pad 12: unconnected-(U103-Pad12) -> Net-(RN103D-R4.2)
- U103 pad 13: unconnected-(U103-Pad13) -> Net-(R106-Pad1)
- U103 pad 2: unconnected-(U103-Pad2) -> Net-(RN101B-R2.2)
- U103 pad 3: unconnected-(U103-Pad3) -> Net-(RN101C-R3.2)
- U103 pad 4: unconnected-(U103-Pad4) -> Net-(RN101D-R4.2)
- U103 pad 5: unconnected-(U103-Pad5) -> Net-(RN102A-R1.2)
- U103 pad 6: unconnected-(U103-Pad6) -> Net-(RN102B-R2.2)
- U103 pad 7: unconnected-(U103-Pad7) -> Net-(RN102C-R3.2)
- U103 pad 8: unconnected-(U103-Pad8) -> Net-(RN102D-R4.2)
- U103 pad 9: unconnected-(U103-Pad9) -> Net-(RN103A-R1.2)
- U104 pad 1: unconnected-(U104-Pad1) -> Net-(RN101A-R1.2)
- U104 pad 10: unconnected-(U104-Pad10) -> Net-(RN103B-R2.2)
- U104 pad 11: unconnected-(U104-Pad11) -> Net-(RN103C-R3.2)
- U104 pad 12: unconnected-(U104-Pad12) -> Net-(RN103D-R4.2)
- U104 pad 13: unconnected-(U104-Pad13) -> Net-(R106-Pad1)
- U104 pad 2: unconnected-(U104-Pad2) -> Net-(RN101B-R2.2)
- U104 pad 3: unconnected-(U104-Pad3) -> Net-(RN101C-R3.2)
- U104 pad 4: unconnected-(U104-Pad4) -> Net-(RN101D-R4.2)
- U104 pad 5: unconnected-(U104-Pad5) -> Net-(RN102A-R1.2)
- U104 pad 6: unconnected-(U104-Pad6) -> Net-(RN102B-R2.2)
- U104 pad 7: unconnected-(U104-Pad7) -> Net-(RN102C-R3.2)
- U104 pad 8: unconnected-(U104-Pad8) -> Net-(RN102D-R4.2)
- U104 pad 9: unconnected-(U104-Pad9) -> Net-(RN103A-R1.2)
Routing:
- net Net-(RN103D-R4.2): track 0.00 -> 68.9 mm, vias 0 -> 1
- net BATT: track 0.00 -> 66.8 mm, vias 0 -> 4
- net Net-(RN103C-R3.2): track 0.00 -> 60.4 mm, vias 0 -> 1
- net Net-(RN101A-R1.2): track 0.00 -> 60.3 mm, vias 0 -> 2
- net LED75: track 0.00 -> 60.2 mm, vias 0 -> 1
- net Net-(RN101B-R2.2): track 0.00 -> 60.1 mm, vias 0 -> 2
- net Net-(RN101C-R3.2): track 0.00 -> 59.4 mm, vias 0 -> 2
- net Net-(RN101D-R4.2): track 0.00 -> 58.9 mm, vias 0 -> 2
- net LED50: track 0.00 -> 57.7 mm, vias 0 -> 2
- net Net-(RN102A-R1.2): track 0.00 -> 56.6 mm, vias 0 -> 2
- net 12V: track 0.00 -> 56.3 mm
- net BQ_ALERT: track 0.00 -> 56.2 mm
- net VCC_3V3: track 0.00 -> 54.5 mm
- net LED100: track 0.00 -> 53.2 mm, vias 0 -> 1
- net LED25: track 0.00 -> 49.2 mm, vias 0 -> 2
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- added copper zone on B.Cu, net GND
- added copper zone on F.Cu, net GND
- added copper zone on In1.Cu, net GND
- added copper zone on In2.Cu, net GND
Other:
- board outline added: 27 x 43 mm
- copper layers 2 -> 4
